File: LaTeX/schematics/fft.sch (KiCad schematic (older format))
At the start: 13 parts

Commit message: siunitx compliance, minor fixes
Parts:
- Ib: value Amperemeter_DC -> Amperometer_DC
Changed lines of the file:
@@
 P 7850 2000
 F 0 "Ib" V 7560 2000 50  0000 C CNN
-F 1 "Amperemeter_DC" V 7651 2000 50  0000 C CNN
+F 1 "Amperometer_DC" V 7651 2000 50  0000 C CNN
 F 2 "" V 7850 2100 50  0001 C CNN
 F 3 "~" V 7850 2100 50  0001 C CNN
